File: hardware/pcb_2026_work/bbb.kicad_pcb (KiCad board)
At the start: 4 copper layers, 55.9 x 84.9 mm, 73 parts, among them J1 Conn_02x14_Odd_Even, J2 Conn_02x20_Odd_Even, J3 FC68131, J4 Inductor L1, J5 Inductor L2, J6 Inductor L3, U1 THS4304, U2 Si5351A-B-GT, U3 TS3A5017, U4 TL972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

Commit message: updated schematic and pcb editor files
Parts:
- U8: footprint Analog switchx2:DGS0010A_N -> TI_Analog_Switch:DGS0010A_N
- moved C33 193.9 mm to (161.3, 111.0)
- moved C34 189.4 mm to (161.3, 106.0), turned to 180 degrees
- moved U8 186.4 mm to (142.8, 136.0), turned to 180 degrees
- moved L4 185.3 mm to (161.3, 114.0), turned to 180 degrees
- moved R22 184.7 mm to (160.3, 101.5), turned to 90 degrees
- moved R23 182.4 mm to (156.8, 106.0)
- moved U7 182.2 mm to (154.6, 111.0)
- moved L5 176.1 mm to (154.8, 114.0)
Connections:
- C8 pad 1: MIXI+ -> MIXQ+
- J1 pad 23: MIXI+ -> MIXQ+
- U3 pad 10: MIXI+ -> MIXQ+
- U3 pad 6: MIXI+ -> MIXQ+
Routing:
- net +5V: track 15.4 -> 78.6 mm
- net GPIO23: track 0.00 -> 58.3 mm, vias 0 -> 2
- net CLK2: track 14.0 -> 44.4 mm
- net TX_RF: track 0.00 -> 30.4 mm, vias 0 -> 2
- net RFIN: track 15.1 -> 44.7 mm
- net GND: track 118.1 -> 142.4 mm, vias 31 -> 33
- net MIXI+: track 45.6 -> 21.9 mm, vias 2 -> 1
- net MIXQ+: track 0.00 -> 23.7 mm, vias 0 -> 1
- net SMA: track 0.00 -> 22.9 mm
- net BPFOUT: track 24.5 -> 46.9 mm, vias 0 -> 2
- net Net-(U7-G): track 0.00 -> 11.5 mm
- net Net-(U7-D): track 0.00 -> 11.3 mm
- net BPFIN: track 43.8 -> 40.6 mm, vias 1 -> 2
