File: hardware/pcb_2026_work/bbb.kicad_sch (KiCad schematic)
At the start: 73 parts, among them J1 Conn_02x14_Odd_Even, J2 Conn_02x20_Odd_Even, J3 FC68131, J4 Inductor L1, J5 Inductor L2, J6 Inductor L3, U1 THS4304, U2 Si5351A-B-GT, U3 TS3A5017, U4 TL972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

Commit message: updated schematic and pcb editor files
Connections:
- net MIXI+: no longer C8.1, J1.23 (Pin_23), U3.10 (2S1), U3.6 (1S1)
- new net MIXQ+: C8.1, J1.23 (Pin_23), U3.10 (2S1), U3.6 (1S1)
Other:
- note added: "12/05/2026"
- note added: "ELEC3607 Software Defined Radio : Transciever"
- note removed: "17/02/2025"
- note removed: "ELEC3607 Software Defined Radio"
- moved on the sheet: C33, C34, C7, D1, D2, L4, L5, R10, R11, R22, R23, U7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
